Commit message: After 10000 hours of debugging :////

File: tbai_description/urdf/anymal_d_gazebo.urdf.xacro (robot description, xacro)
@@ -32,3 +32,308 @@
   <plugin filename="libStatePublisher.so" name="StatePublisher"/>
 </gazebo>
+ <joint name="face_front_to_depth_camera_front_camera" type="fixed">
+        <parent link="face_front"/>
+        <child link="depth_camera_front_camera"/>
+        <origin rpy="0.0 0.523598775598 0" xyz="0.04715 0.0 -0.0292"/>
+    </joint>
+    <!-- Camera link -->
+    <link name="depth_camera_front_camera">
+        <inertial>
+            <origin rpy="0 0 0" xyz="-0.021 -0.002 0.025"/>
+            <mass value="0.16043"/>
+            <inertia ixx="0.000637051" ixy="0.000484569" ixz="0.000424211" iyy="0.000929402" iyz="5.138e-06" izz="0.000484569"/>
+        </inertial>
+    </link>
+    <!-- Camera parent joint -->
+    <!-- Frame lies on the left ir camera according to any_realsense2_camera urdf. -->
+    <joint name="depth_camera_front_camera_to_camera_parent" type="fixed">
+        <parent link="depth_camera_front_camera"/>
+        <child link="depth_camera_front_camera_parent"/>
+        <origin rpy="0.0 0.0 0.0" xyz="0.0255 0.0175 0.0"/>
+    </joint>
+    <!-- Camera parent link -->
+    <link name="depth_camera_front_camera_parent"/>
+    <!-- Depth optical frame joint -->
+    <joint name="depth_camera_front_camera_parent_to_depth_optical_frame" type="fixed">
+        <parent link="depth_camera_front_camera_parent"/>
+        <child link="depth_camera_front_depth_optical_frame"/>
+        <origin rpy="-1.57079632679 0.0 -1.57079632679" xyz="0.0 0.0 0.0"/>
+    </joint>
+    <!-- Depth optical frame link -->
+    <link name="depth_camera_front_depth_optical_frame"/>
+    <!-- Camera color frame joint -->
+    <joint name="depth_camera_front_camera_parent_to_color_frame" type="fixed">
+        <parent link="depth_camera_front_camera_parent"/>
+        <child link="depth_camera_front_color_frame"/>
+        <origin rpy="0 0 0" xyz="0 0.015 0"/>
+    </joint>
+    <!-- Camera color frame link -->
+    <link name="depth_camera_front_color_frame"/>
+    <!-- Camera color optical joint -->
+    <joint name="depth_camera_front_color_frame_to_color_optical_frame" type="fixed">
+        <parent link="depth_camera_front_color_frame"/>
+        <child link="depth_camera_front_color_optical_frame"/>
+        <origin rpy="-1.57079632679 0.0 -1.57079632679" xyz="0.0 0.0 0.0"/>
+    </joint>
+    <!-- Camera color optical link -->
+    <link name="depth_camera_front_color_optical_frame"/>
+    <!-- Camera joint -->
+    <!-- Is located in the center of the mounting points. -->
+     <!-- Camera joint -->
+    <!-- Is located between the two back screw holes at ground level. -->
+    <joint name="face_rear_to_depth_camera_rear_camera" type="fixed">
+        <parent link="face_rear"/>
+        <child link="depth_camera_rear_camera"/>
+        <origin rpy="0.0 0.523598775598 0" xyz="0.04715 0.0 -0.0292"/>
+    </joint>
+    <!-- Camera link -->
+    <link name="depth_camera_rear_camera">
+        <inertial>
+            <origin rpy="0 0 0" xyz="-0.021 -0.002 0.025"/>
+            <mass value="0.16043"/>
+            <inertia ixx="0.000637051" ixy="0.000484569" ixz="0.000424211" iyy="0.000929402" iyz="5.138e-06" izz="0.000484569"/>
+        </inertial>
+    </link>
+    <!-- Camera parent joint -->
+    <!-- Frame lies on the left ir camera according to any_realsense2_camera urdf. -->
+    <joint name="depth_camera_rear_camera_to_camera_parent" type="fixed">
+        <parent link="depth_camera_rear_camera"/>
+        <child link="depth_camera_rear_camera_parent"/>
+        <origin rpy="0.0 0.0 0.0" xyz="0.0255 0.0175 0.0"/>
+    </joint>
+    <!-- Camera parent link -->
+    <link name="depth_camera_rear_camera_parent"/>
+    <!-- Depth optical frame joint -->
+    <joint name="depth_camera_rear_camera_parent_to_depth_optical_frame" type="fixed">
+        <parent link="depth_camera_rear_camera_parent"/>
+        <child link="depth_camera_rear_depth_optical_frame"/>
+        <origin rpy="-1.57079632679 0.0 -1.57079632679" xyz="0.0 0.0 0.0"/>
+    </joint>
+    <!-- Depth optical frame link -->
+    <link name="depth_camera_rear_depth_optical_frame"/>
+    <!-- Camera color frame joint -->
+    <joint name="depth_camera_rear_camera_parent_to_color_frame" type="fixed">
+        <parent link="depth_camera_rear_camera_parent"/>
+        <child link="depth_camera_rear_color_frame"/>
+        <origin rpy="0 0 0" xyz="0 0.015 0"/>
+    </joint>
+    <!-- Camera color frame link -->
+    <link name="depth_camera_rear_color_frame"/>
+    <!-- Camera color optical joint -->
+    <joint name="depth_camera_rear_color_frame_to_color_optical_frame" type="fixed">
+        <parent link="depth_camera_rear_color_frame"/>
+        <child link="depth_camera_rear_color_optical_frame"/>
+        <origin rpy="-1.57079632679 0.0 -1.57079632679" xyz="0.0 0.0 0.0"/>
+    </joint>
+    <!-- Camera color optical link -->
+    <link name="depth_camera_rear_color_optical_frame"/>
+    <!-- Camera joint -->
+  <!-- Front camera -->
+<!-- Front depth camera -->
+<gazebo reference="depth_camera_front_camera">
+<sensor type="depth" name="realsense_R200">
+    <always_on>true</always_on>
+    <visualize>false</visualize>
+    <update_rate>3</update_rate>
+    <camera>
+        <horizontal_fov>2.0</horizontal_fov>
+        <image>
+            <width>640</width>
+            <height>480</height>
+            <format>R8G8B8</format>
+        </image>
+        <depth_camera></depth_camera>
+        <clip>
+            <near>0.2</near>
+            <far>3</far>
+        </clip>
+        <noise>
+          <type>gaussian</type>
+          <mean>0.0</mean>
+          <stddev>0.05</stddev>
+        </noise>
+    </camera>
+    <plugin name="camera_controller" filename="libgazebo_ros_openni_kinect.so">
+    <baseline>0.2</baseline>
+    <alwaysOn>true</alwaysOn>
+    <updateRate>0.0</updateRate>
+    <cameraName>camera</cameraName>
+    <frameName>depth_camera_front_depth_optical_frame</frameName>
+    <imageTopicName>rgb/image_raw</imageTopicName>
+    <depthImageTopicName>depth/image_raw</depthImageTopicName>
+    <pointCloudTopicName>depth/points</pointCloudTopicName>
+    <cameraInfoTopicName>rgb/camera_info</cameraInfoTopicName>
+    <depthImageCameraInfoTopicName>depth/camera_info</depthImageCameraInfoTopicName>
+    <pointCloudCutoff>0.4</pointCloudCutoff>
+    <pointCloudCutoffMax>3.0</pointCloudCutoffMax>
+        <hackBaseline>0.07</hackBaseline>
+        <distortionK1>0.0</distortionK1>
+        <distortionK2>0.0</distortionK2>
+        <distortionK3>0.0</distortionK3>
+        <distortionT1>0.0</distortionT1>
+        <distortionT2>0.0</distortionT2>
+    <CxPrime>0.0</CxPrime>
+    <Cx>0.0</Cx>
+    <Cy>0.0</Cy>
+    <focalLength>0</focalLength>
+    <hackBaseline>0</hackBaseline>
+    </plugin>
+</sensor>
+</gazebo>
+<!-- Back camera -->
+<!-- Back depth camera -->
+<gazebo reference="depth_camera_rear_camera">
+<sensor type="depth" name="realsense_R200">
+    <always_on>true</always_on>
+    <visualize>false</visualize>
+    <update_rate>3</update_rate>
+    <camera>
+        <horizontal_fov>2.0</horizontal_fov>
+        <image>
+            <width>640</width>
+            <height>480</height>
+            <format>R8G8B8</format>
+        </image>
+        <depth_camera></depth_camera>
+        <clip>
+            <near>0.2</near>
+            <far>3</far>
+        </clip>
+        <noise>
+          <type>gaussian</type>
+          <mean>0.0</mean>
+          <stddev>0.05</stddev>
+        </noise>
+    </camera>
+    <plugin name="camera_controller" filename="libgazebo_ros_openni_kinect.so">
+    <baseline>0.2</baseline>
+    <alwaysOn>true</alwaysOn>
+    <updateRate>0.0</updateRate>
+    <cameraName>rear_camera</cameraName>
+    <frameName>depth_camera_rear_depth_optical_frame</frameName>
+    <imageTopicName>rgb/image_raw</imageTopicName>
+    <depthImageTopicName>depth/image_raw</depthImageTopicName>
+    <pointCloudTopicName>depth/points</pointCloudTopicName>
+    <cameraInfoTopicName>rgb/camera_info</cameraInfoTopicName>
+    <depthImageCameraInfoTopicName>depth/camera_info</depthImageCameraInfoTopicName>
+    <pointCloudCutoff>0.4</pointCloudCutoff>
+    <pointCloudCutoffMax>3.0</pointCloudCutoffMax>
+        <hackBaseline>0.07</hackBaseline>
+        <distortionK1>0.0</distortionK1>
+        <distortionK2>0.0</distortionK2>
+        <distortionK3>0.0</distortionK3>
+        <distortionT1>0.0</distortionT1>
+        <distortionT2>0.0</distortionT2>
+    <CxPrime>0.0</CxPrime>
+    <Cx>0.0</Cx>
+    <Cy>0.0</Cy>
+    <focalLength>0</focalLength>
+    <hackBaseline>0</hackBaseline>
+    </plugin>
+</sensor>
+</gazebo>
+<!-- Left camera -->
+<!-- Left depth camera -->
+<gazebo reference="depth_camera_left_camera">
+<sensor type="depth" name="realsense_R200">
+    <always_on>true</always_on>
+    <visualize>false</visualize>
+    <update_rate>3</update_rate>
+    <camera>
+        <horizontal_fov>2.0</horizontal_fov>
+        <image>
+            <width>640</width>
+            <height>480</height>
+            <format>R8G8B8</format>
+        </image>
+        <depth_camera></depth_camera>
+        <clip>
+            <near>0.2</near>
+            <far>3</far>
+        </clip>
+        <noise>
+          <type>gaussian</type>
+          <mean>0.0</mean>
+          <stddev>0.05</stddev>
+        </noise>
+    </camera>
+    <plugin name="camera_controller" filename="libgazebo_ros_openni_kinect.so">
+    <baseline>0.2</baseline>
+    <alwaysOn>true</alwaysOn>
+    <updateRate>0.0</updateRate>
+    <cameraName>left_camera</cameraName>
+    <frameName>depth_camera_left_depth_optical_frame</frameName>
+    <imageTopicName>rgb/image_raw</imageTopicName>
+    <depthImageTopicName>depth/image_raw</depthImageTopicName>
+    <pointCloudTopicName>depth/points</pointCloudTopicName>
+    <cameraInfoTopicName>rgb/camera_info</cameraInfoTopicName>
+    <depthImageCameraInfoTopicName>depth/camera_info</depthImageCameraInfoTopicName>
+    <pointCloudCutoff>0.4</pointCloudCutoff>
+    <pointCloudCutoffMax>3.0</pointCloudCutoffMax>
+        <hackBaseline>0.07</hackBaseline>
+        <distortionK1>0.0</distortionK1>
+        <distortionK2>0.0</distortionK2>
+        <distortionK3>0.0</distortionK3>
+        <distortionT1>0.0</distortionT1>
+        <distortionT2>0.0</distortionT2>
+    <CxPrime>0.0</CxPrime>
+    <Cx>0.0</Cx>
+    <Cy>0.0</Cy>
+    <focalLength>0</focalLength>
+    <hackBaseline>0</hackBaseline>
+    </plugin>
+</sensor>
+</gazebo>
+<!-- Right camera -->
+<!-- Right depth camera -->
+<gazebo reference="depth_camera_right_camera">
+<sensor type="depth" name="realsense_R200">
+    <always_on>true</always_on>
+    <visualize>false</visualize>
+    <update_rate>3</update_rate>
+    <camera>
+        <horizontal_fov>2.0</horizontal_fov>
+        <image>
+            <width>640</width>
+            <height>480</height>
+            <format>R8G8B8</format>
+        </image>
+        <depth_camera></depth_camera>
+        <clip>
+            <near>0.2</near>
+            <far>3</far>
+        </clip>
+        <noise>
+          <type>gaussian</type>
+          <mean>0.0</mean>
+          <stddev>0.05</stddev>
+        </noise>
+    </camera>
+    <plugin name="camera_controller" filename="libgazebo_ros_openni_kinect.so">
+    <baseline>0.2</baseline>
+    <alwaysOn>true</alwaysOn>
+    <updateRate>0.0</updateRate>
+    <cameraName>right_camera</cameraName>
+    <frameName>depth_camera_right_depth_optical_frame</frameName>
+    <imageTopicName>rgb/image_raw</imageTopicName>
+    <depthImageTopicName>depth/image_raw</depthImageTopicName>
+    <pointCloudTopicName>depth/points</pointCloudTopicName>
+    <cameraInfoTopicName>rgb/camera_info</cameraInfoTopicName>
+    <depthImageCameraInfoTopicName>depth/camera_info</depthImageCameraInfoTopicName>
+    <pointCloudCutoff>0.4</pointCloudCutoff>
+    <pointCloudCutoffMax>3.0</pointCloudCutoffMax>
+        <hackBaseline>0.07</hackBaseline>
+        <distortionK1>0.0</distortionK1>
+        <distortionK2>0.0</distortionK2>
+        <distortionK3>0.0</distortionK3>
+        <distortionT1>0.0</distortionT1>
+        <distortionT2>0.0</distortionT2>
+    <CxPrime>0.0</CxPrime>
+    <Cx>0.0</Cx>
+    <Cy>0.0</Cy>
+    <focalLength>0</focalLength>
+    <hackBaseline>0</hackBaseline>
+    </plugin>
+</sensor>
+</gazebo>
 </robot>

Commit message: Add contact sensors

File: tbai_description/urdf/anymal_d_gazebo.urdf.xacro (robot description, xacro)
@@ -337,3 +337,36 @@
 </sensor>
 </gazebo>
+<!-- Add contact sensors -->
+<gazebo reference="LF_FOOT">
+    <sensor name="lf_foot_contact" type="contact">
+    <plugin name="lf_contact_plugin" filename="libContactSensor.so"/>
+    <contact>
+        <collision>LF_SHANK_fixed_joint_lump__LF_FOOT_collision_3</collision>
+    </contact>
+    </sensor>
+</gazebo>
+<gazebo reference="RF_FOOT">
+    <sensor name="rf_foot_contact" type="contact">
+    <plugin name="rf_contact_plugin" filename="libContactSensor.so"/>
+    <contact>
+        <collision>RF_SHANK_fixed_joint_lump__RF_FOOT_collision_3</collision>
+    </contact>
+    </sensor>
+</gazebo>
+<gazebo reference="LH_FOOT">
+    <sensor name="lh_foot_contact" type="contact">
+    <plugin name="lh_contact_plugin" filename="libContactSensor.so"/>
+    <contact>
+        <collision>LH_SHANK_fixed_joint_lump__LH_FOOT_collision_3</collision>
+    </contact>
+    </sensor>
+</gazebo>
+<gazebo reference="RH_FOOT">
+    <sensor name="rh_foot_contact" type="contact">
+    <plugin name="rh_contact_plugin" filename="libContactSensor.so"/>
+    <contact>
+        <collision>RH_SHANK_fixed_joint_lump__RH_FOOT_collision_3</collision>
+    </contact>
+    </sensor>
+</gazebo>
 </robot>
